File: kicad-gps-shield.kicad_pcb (KiCad board)
At the start: 2 copper layers, 65 x 62.1 mm, 34 parts, among them J1 FTDI, J2 FTDI, J3 USB_B_Micro, P1 Conn_02x20_Odd_Even, U1 GNSS_RTK_Click, U2 HC-12, U3 NS-HP, U4 HC-12, U5 Sparkfun-Zed-F9P, U6 Navspark_Mini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

Commit message: V2
Parts:
- removed JP2, JP4: SolderJumper_2_Open, Jumper:SolderJumper-2_P1.3mm_Open_Pad1.0x1.5mm
- removed JP3: SolderJumper_2_Bridged, Jumper:SolderJumper-2_P1.3mm_Bridged_Pad1.0x1.5mm
- removed REF**: OSHW-Logo2_7.3x6mm_SilkScreen, Symbol:OSHW-Logo2_7.3x6mm_SilkScreen
- removed REF**: Symbol_Danger_CopperTop_Small, Symbol:Symbol_Danger_CopperTop_Small
- removed REF**: OSHW-Symbol_44.5x40mm_SilkScreen, Symbol:OSHW-Symbol_44.5x40mm_SilkScreen
- removed REF**: KiCad-Logo_5mm_SilkScreen, Symbol:KiCad-Logo_5mm_SilkScreen
- removed U1: GNSS_RTK_Click, Modules:GNSS RTK Click
- removed U7: Navspark_Uart, Modules:Navspark Uart
- added H1: SMA, MountingHole:MountingHole_6.4mm_M6_ISO14580, F.Cu at (169.5, 132.2)
- added J10: GNSS U2, Connector_PinSocket_2.54mm:PinSocket_1x02_P2.54mm_Vertical, F.Cu at (189.9, 97.8)
- added J11: Serial 2, Connector_PinSocket_2.54mm:PinSocket_1x02_P2.54mm_Vertical, F.Cu at (189.8, 123.3)
- added J4: Oled, Connector_PinSocket_2.54mm:PinSocket_1x04_P2.54mm_Vertical, F.Cu at (153.7, 128.4)
- added J5: RTC, Connector_PinSocket_2.54mm:PinSocket_2x05_P2.54mm_Vertical, B.Cu at (147.9, 125.9)
- added J6: UART2, Connector_PinSocket_2.54mm:PinSocket_1x02_P2.54mm_Vertical, F.Cu at (193.2, 86.1)
- added J7: UART3, Connector_PinSocket_2.54mm:PinSocket_1x02_P2.54mm_Vertical, F.Cu at (197.4, 86.1)
- added J8: UART4, Connector_PinSocket_2.54mm:PinSocket_1x02_P2.54mm_Vertical, F.Cu at (188.6, 86.1)
- added J9: UART5, Connector_PinSocket_2.54mm:PinSocket_1x02_P2.54mm_Vertical, F.Cu at (201.7, 86.1)
- added JP5: 3V<>GND, Jumper:SolderJumper-3_P2.0mm_Open_TrianglePad1.0x1.5mm, F.Cu at (186.5, 128.4)
- added JP6: Pi 3V3, Jumper:SolderJumper-2_P1.3mm_Open_TrianglePad1.0x1.5mm, B.Cu at (171.9, 87.5)
- added JP7: Pi 5V, Jumper:SolderJumper-2_P1.3mm_Open_TrianglePad1.0x1.5mm, B.Cu at (151.0, 84.3)
- added R5: R_Small, Resistor_SMD:R_0805_2012Metric_Pad1.20x1.40mm_HandSolder, F.Cu at (151.7, 95.0)
- added R6: R_Small, Resistor_SMD:R_0805_2012Metric_Pad1.20x1.40mm_HandSolder, F.Cu at (151.7, 99.2)
- added TP1: TestPoint, TestPoint:TestPoint_THTPad_2.5x2.5mm_Drill1.2mm, F.Cu at (182.7, 131.8)
- added TP2: TestPoint, TestPoint:TestPoint_THTPad_2.5x2.5mm_Drill1.2mm, F.Cu at (190.6, 131.8)
- C1, C2, U8: moved to B.Cu
- J3: value USB_B_Micro -> Power IN; footprint Connector_USB:USB_Micro-B_Amphenol_10118194_Horizontal -> Connector_PinSocket_2.54mm:PinSocket_1x02_P2.54mm_Vertical
- JP1: value SolderJumper_2_Open -> 3V3<>5V; footprint Jumper:SolderJumper-2_P1.3mm_Open_Pad1.0x1.5mm -> Jumper:SolderJumper-3_P2.0mm_Open_TrianglePad1.0x1.5mm; moved to B.Cu
- moved D2 60.0 mm to (188.9, 135.3), turned to 0 degrees
- moved D1 58.9 mm to (184.9, 135.3), turned to 180 degrees
- moved R1 54.5 mm to (185.6, 132.0), turned to -90 degrees
- moved R2 54.1 mm to (187.7, 132.0), turned to -90 degrees
- moved JP1 48.7 mm to (145.4, 87.1), turned to 90 degrees
- moved J3 47.5 mm to (142.8, 88.4), turned to 180 degrees
- moved C1 32.8 mm to (166.7, 90.7), turned to 180 degrees
- moved U8 28.4 mm to (166.7, 102.6)
- moved C2 25.2 mm to (166.7, 95.8)
- moved U6 8.69 mm to (165.7, 118.2), turned to 0 degrees
- moved D4 8.59 mm to (197.2, 135.3), turned to 0 degrees
- moved D3 7.82 mm to (193.0, 135.3), turned to 180 degrees
- moved R3 7.34 mm to (194.0, 132.3)
- moved U5 6.56 mm to (158.1, 100.5), turned to -90 degrees
- moved R4 4.66 mm to (196.3, 132.3)
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Connections:
- J2 pad 4: GPS RX2 -> Serial2TX
- J2 pad 5: GPS TX2 -> Serial2RX
- J3 pad 1: +5V -> Net-(J3-Pad1)
- J3 pad 2: unconnected-(J3-Pad2) -> GND
- JP1 pad 1: /GPIO12(PWM0) -> +3V3
- JP1 pad 2: GPS RX2 -> Net-(J3-Pad1)
- P1 pad 1: +3V3 -> Net-(P1-Pad1)
- P1 pad 16: /GPIO23(GEN4) -> PI-TX3
- P1 pad 17: +3V3 -> Net-(P1-Pad1)
- P1 pad 2: +5V -> Net-(P1-Pad2)
- P1 pad 21: /GPIO9(SPI0_MISO) -> PI-RX4
- P1 pad 24: /GPIO8(SPI0_CE_N) -> PI-TX4
- P1 pad 27: /ID_SD -> PI-TX2
- P1 pad 28: /ID_SC -> PI-RX2
- P1 pad 29: /GPIO5 -> PI-RX3
- P1 pad 32: /GPIO12(PWM0) -> PI-TX5
- P1 pad 33: /GPIO13(PWM1) -> PI-RX5
- P1 pad 4: +5V -> Net-(P1-Pad2)
- R1 pad 1: GND -> Net-(JP5-Pad2)
- R2 pad 1: GND -> Net-(JP5-Pad2)
- U4 pad 3: GPS TX2 -> Serial2RX
- U4 pad 4: GPS RX2 -> Serial2TX
- U5 pad 12: Net-(JP4-Pad2) -> unconnected-(U5-Pad12)
- U5 pad 13: Net-(JP3-Pad2) -> +3V3
- U6 pad 11: SCL -> unconnected-(U6-Pad11)
- U6 pad 2: SDA -> unconnected-(U6-Pad2)
Routing:
- net GPS RX2: track 119.4 -> 11.1 mm, vias 2 -> 0
- net GPS TX2: track 115.7 -> 18.4 mm, vias 2 -> 0
- net +3V3: track 182.7 -> 252.7 mm
- net +5V: track 143.2 -> 91.9 mm, vias 4 -> 3
- net PPS: track 88.9 -> 131.6 mm, vias 3 -> 0
- net Net-(P1-Pad1): track 0.00 -> 39.3 mm
- net PI-TX3: track 0.00 -> 37.0 mm
- net GPS TX1: track 116.2 -> 94.8 mm, vias 4 -> 0
- net PI-RX2: track 0.00 -> 19.9 mm
- net PI-TX5: track 0.00 -> 19.4 mm
- net PI-RX3: track 0.00 -> 17.9 mm
- net PI-RX4: track 0.00 -> 17.2 mm
- net PI-RX5: track 0.00 -> 16.7 mm
- net SDA: track 45.1 -> 61.8 mm, vias 2 -> 1
- net PI-TX4: track 0.00 -> 16.0 mm
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Other:
- board text added: "5V 3V3"
- board text added: "GPS Shiels v2"
- board text added: "I2C Pullup"
- board text added: "PI Uarts"
- board text added: "RX TX"
- board text added: "TX RX"
- board text removed: "GPS Shiels v1"
- board text removed: "Select Sparkfun Power 3v3 or 5V"
