File: kicad-gps-shield.kicad_sch (KiCad schematic)
At the start: 31 parts, among them J1 FTDI, J2 FTDI, J3 USB_B_Micro, P1 Conn_02x20_Odd_Even, U1 GNSS_RTK_Click, U2 HC-12, U3 NS-HP, U4 HC-12, U5 Sparkfun-Zed-F9P, U6 Navspark_Mini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

Commit message: V2
Parts:
- removed A1: Arduino_Leonardo, Modules:Arduino_UNO_R3, symbol MCU_Module:Arduino_Leonardo
- removed J3: USB_B_Micro, Connector_USB:USB_Micro-B_Amphenol_10118194_Horizontal, symbol Connector:USB_B_Micro
- removed JP1, JP2, JP4: SolderJumper_2_Open, Jumper:SolderJumper-2_P1.3mm_Bridged2Bar_Pad1.0x1.5mm, symbol Jumper:SolderJumper_2_Open
- removed JP3: SolderJumper_2_Bridged, Jumper:SolderJumper-2_P1.3mm_Bridged_Pad1.0x1.5mm, symbol Jumper:SolderJumper_2_Bridged
- removed U1: GNSS_RTK_Click, Modules:GNSS RTK Click, symbol Modules:GNSS_RTK_Click
- removed U7: Navspark_Uart, Modules:Navspark Uart, symbol Modules:Navspark_Uart
- added H1: SMA, MountingHole:MountingHole_6.4mm_M6_ISO14580, symbol Mechanical:MountingHole
- added J10: GNSS U2, Connector_PinSocket_2.54mm:PinSocket_1x02_P2.54mm_Vertical, symbol Connector_Generic:Conn_01x02
- added J11: Serial 2, Connector_PinSocket_2.54mm:PinSocket_1x02_P2.54mm_Vertical, symbol Connector_Generic:Conn_01x02
- added J3: Power IN, Connector_PinSocket_2.54mm:PinSocket_1x02_P2.54mm_Vertical, symbol Connector:Screw_Terminal_01x02
- added J4: Oled, Connector_PinSocket_2.54mm:PinSocket_1x04_P2.54mm_Vertical, symbol Connector:Conn_01x04_Female
- added J5: RTC, Connector_PinSocket_2.54mm:PinSocket_2x05_P2.54mm_Vertical, symbol Connector_Generic:Conn_02x05_Odd_Even
- added J6: UART2, Connector_PinSocket_2.54mm:PinSocket_1x02_P2.54mm_Vertical, symbol Connector_Generic:Conn_01x02
- added J7: UART3, Connector_PinSocket_2.54mm:PinSocket_1x02_P2.54mm_Vertical, symbol Connector_Generic:Conn_01x02
- added J8: UART4, Connector_PinSocket_2.54mm:PinSocket_1x02_P2.54mm_Vertical, symbol Connector_Generic:Conn_01x02
- added J9: UART5, Connector_PinSocket_2.54mm:PinSocket_1x02_P2.54mm_Vertical, symbol Connector_Generic:Conn_01x02
- added JP1: 3V3<>5V, Jumper:SolderJumper-3_P2.0mm_Open_TrianglePad1.0x1.5mm, symbol Jumper:SolderJumper_3_Open
- added JP5: 3V<>GND, Jumper:SolderJumper-3_P2.0mm_Open_TrianglePad1.0x1.5mm, symbol Jumper:SolderJumper_3_Open
- added JP6: Pi 3V3, Jumper:SolderJumper-2_P1.3mm_Open_TrianglePad1.0x1.5mm, symbol Jumper:SolderJumper_2_Open
- added JP7: Pi 5V, Jumper:SolderJumper-2_P1.3mm_Open_TrianglePad1.0x1.5mm, symbol Jumper:SolderJumper_2_Open
- added R5, R6: R_Small, Resistor_SMD:R_0805_2012Metric_Pad1.20x1.40mm_HandSolder, symbol Device:R_Small
- added TP1, TP2: TestPoint, TestPoint:TestPoint_THTPad_2.5x2.5mm_Drill1.2mm, symbol Connector:TestPoint
Connections:
- net +3V3: now also U5.13 (VCC33), J4.3 (Pin_3), J5.1 (Pin_1), JP1.1 (A), JP5.1 (A), JP6.1 (A), R5.1, R6.1; no longer P1.1 (Pin_1), P1.17 (Pin_17)
- net +5V: now also JP1.3 (B), JP7.2 (B); no longer P1.2 (Pin_2), P1.4 (Pin_4)
- net GND: now also J3.2 (Pin_2), J4.4 (Pin_4), J5.6 (Pin_6), J5.9 (Pin_9), JP5.3 (B); no longer R1.1, R2.1
- net GPS RX2: now also J10.2 (Pin_2); no longer J2.4 (TXD), U4.4 (TXD)
- net GPS TX2: now also J10.1 (Pin_1); no longer J2.5 (RXD), U4.3 (RXD)
- net PPS: now also TP2.1
- net RTK: now also TP1.1
- net SCL: now also J4.2 (Pin_2), J5.5 (Pin_5), R6.2; no longer U6.11 (SCL)
- net SDA: now also J4.1 (Pin_1), J5.3 (Pin_3), R5.2; no longer U6.2 (SDA)
- net GPIO12(PWM0) renamed PI-TX5
- net PI-TX5: now also J9.1 (Pin_1)
- net GPIO13(PWM1) renamed PI-RX5
- net PI-RX5: now also J9.2 (Pin_2)
- net GPIO23(GEN4) renamed PI-TX3
- net PI-TX3: now also J7.1 (Pin_1)
- net GPIO5 renamed PI-RX3
- net PI-RX3: now also J7.2 (Pin_2)
- net GPIO8(SPI0_CE_N) renamed PI-TX4
- net PI-TX4: now also J8.1 (Pin_1)
- net GPIO9(SPI0_MISO) renamed PI-RX4
- net PI-RX4: now also J8.2 (Pin_2)
- net ID_SC renamed PI-RX2
- net PI-RX2: now also J6.2 (Pin_2)
- net ID_SD renamed PI-TX2
- net PI-TX2: now also J6.1 (Pin_1)
- new net: JP6.2 (B), P1.1 (Pin_1), P1.17 (Pin_17)
- new net: JP7.1 (A), P1.2 (Pin_2), P1.4 (Pin_4)
- new net: JP5.2 (C), R1.1, R2.1
- new net: J3.1 (Pin_1), JP1.2 (C)
- new net Serial2RX: J11.2 (Pin_2), J2.5 (RXD), U4.3 (RXD)
- new net Serial2TX: J11.1 (Pin_1), J2.4 (TXD), U4.4 (TXD)
- no-connect marks 4 -> 0
Other:
- moved on the sheet: D3, R3
